File: hardware/electronics/PCBs/Mini_KiCAD/MCU.kicad_sch (KiCad schematic)
At the start: 13 parts, among them J3 HEADER2, U1 ATMEGA32U4RC-AU

Commit message: Initial commit of the PCB project file replacing the ADNS-5050 with PMW3360, referencing the schematic of the Ploopy Classic.
Parts:
- added MCU.C.2, MCU.C.3: 0805, Chip_Passives.PcbLib:0805 - TALL, symbol Mini-altium-import:MCU_1_Cap 0.1uF 100V
- added MCU.J.1: ~, Connectors.PcbLib:6x2, symbol Mini-altium-import:MCU_0_Atmel_ICSP
- MCU.C.1, MCU.C.22, MCU.C.4, MCU.C.5, MCU.C.6, MCU.C.7, MCU.C.8, MCU.C.9: footprint 0805 - TALL -> Chip_Passives.PcbLib:0805 - TALL
- MCU.J.3: renamed from J3; footprint 2x1 -> Connectors.PcbLib:2x1
- MCU.R.1, MCU.R.5: footprint 0805 -> Chip_Passives.PcbLib:0805
- MCU.U.1: renamed from U1; footprint ATmega32U4 - TQFP80P1200X1200X120-44N -> MCUs.PcbLib:ATmega32U4 - TQFP80P1200X1200X120-44N
- MCU.Y.1: footprint LFXTAL055663BULK -> Crystals.PcbLib:LFXTAL055663BULK
Connections:
- net ADNS_SCLK is gone; now on net GND: MCU.U.1.12 (PB7_(PCINT7/OC0A/OC1C/~{RTS}))
- net ADNS_SDIO is gone; now on net GND: MCU.U.1.31 (PC6_(OC3A/~{OC4A}))
- net ADNS_~{CS} is gone; now on net GND: MCU.U.1.28 (PB4_(PCINT4/ADC11))
- net GND: now also MCU.C.2.1, MCU.C.3.1, MCU.J.1.6 (GND); no longer MCU.U.1.19 (PD1_(SDA/INT1)), MCU.U.1.8 (PB0_(SS/PCINT0))
- net MISO: now also MCU.J.1.1 (MISO)
- net MOSI: now also MCU.J.1.4 (MOSI)
- net SCLK: now also MCU.J.1.3 (SCK)
- net V_USB: no longer MCU.C.5.2, MCU.C.6.2, MCU.C.7.2, MCU.C.8.2, MCU.C.9.2, MCU.R.1.2, MCU.R.5.2, MCU.U.1.14 (VCC), MCU.U.1.24 (AVCC), MCU.U.1.34 (VCC), MCU.U.1.44 (AVCC)
- net ~{RESET}: now also MCU.J.1.5 (RST)
- net at MCU.U.1.16 (XTAL2), MCU.Y.1.1: now also MCU.C.3.2
- net at MCU.U.1.17 (XTAL1), MCU.Y.1.3: now also MCU.C.2.2
- new net 3V3: MCU.C.5.2, MCU.C.6.2, MCU.C.7.2, MCU.C.8.2, MCU.C.9.2, MCU.J.1.2 (5V), MCU.R.1.2, MCU.R.5.2, MCU.U.1.14 (VCC), MCU.U.1.24 (AVCC), MCU.U.1.34 (VCC), MCU.U.1.44 (AVCC)
- new net MOTION: MCU.U.1.19 (PD1_(SDA/INT1))
- new net ~{CS}: MCU.U.1.8 (PB0_(SS/PCINT0))
- no-connect marks 1 -> 0
